File: PottyBox4.kicad_pcb (KiCad board)
At the start: 2 copper layers, 51 x 63.5 mm, 52 parts, among them IC1 ESP32-WROVER-B, J1 Sensor 1, J10 Flush 2, J2 Touch 1, J3 Sensor 2, J4 Touch 2, J5 Qwiic, J6 24VAC, J7 DEGUG, J8 Exhaust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

Commit message: Optimize layout, cleanup
Parts:
- moved J4 7.31 mm to (95.0, 80.2)
- moved J2 7.25 mm to (95.0, 72.9)
- moved D8 5.61 mm to (103.2, 107.8)
- moved R13 5.61 mm to (106.8, 107.8)
- moved R12 5.58 mm to (113.6, 107.8)
- moved R15 3.91 mm to (124.2, 106.6), turned to 180 degrees
- moved D9 3.48 mm to (127.7, 103.6), turned to 90 degrees
- moved R14 2.57 mm to (124.2, 102.6), turned to 180 degrees
- moved K3 2.11 mm to (103.2, 104.2)
- moved R16 1.71 mm to (124.2, 104.6), turned to 180 degrees
Connections:
- IC1 pad 8: /TOUCH2 -> /TOUCH1
- IC1 pad 9: /TOUCH1 -> /TOUCH2
Routing:
- net /TOUCH1: track 15.5 -> 23.7 mm
- net /24VAC1: track 55.6 -> 48.4 mm, vias 1 -> 2
- net /EXHAUST: track 14.3 -> 19.7 mm
- net /EN: track 48.2 -> 44.1 mm
- net /LED_SB: track 17.4 -> 20.6 mm
- net /LED_SR: track 22.4 -> 19.2 mm
- net GND: track 51.3 -> 53.9 mm
- net /24VAC2: track 56.2 -> 54.7 mm
- net Net-(J8-Pad1): track 21.4 -> 20.1 mm
- net /SDA: track 38.1 -> 36.9 mm
- net /INT2: track 13.1 -> 11.9 mm
- net Net-(C1-Pad1): track 22.4 -> 21.4 mm
- net +3V3: track 34.4 -> 35.2 mm
- net Net-(J8-Pad2): track 6.49 -> 7.05 mm
Other:
- board text added: "Qwiic"
- board text added: "Sensor 1"
- board text added: "Sensor 2"

Commit message: Final touches
Other:
- board text added: "(c) 2020 Kevin Abraham"
- board text added: ".0"
- board text added: "4.0"
- board text added: "JLCJLCJLCJLC"
- board text added: "PottyBox"
