File: PottyBox4.kicad_pcb (KiCad board)
At the start: 2 copper layers, 51 x 63.5 mm, 52 parts, among them IC1 ESP32-WROVER-B, J1 Sensor 1, J10 Flush 2, J2 Touch 1, J3 Sensor 2, J4 Touch 2, J5 Qwiic, J6 24VAC, J7 DEGUG, J8 Exhaust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

Commit message: Final review and modifications (thanks @tarasjg)
Parts:
- moved J7 3.52 mm to (131.2, 99.7), turned to 45 degrees
Routing:
- net /IO15: track 10.5 -> 7.55 mm
- net GND: track 53.9 -> 51.4 mm, vias 19 -> 17

Commit message: Update to work with KiCad pre-6
Parts:
- C2, C3, C4, C5: footprint Capacitor_SMD:C_0603_1608Metric_Pad1.05x0.95mm_HandSolder -> Capacitor_SMD:C_0603_1608Metric_Pad1.08x0.95mm_HandSolder
- R1, R10, R11, R12, R13, R14, R15, R16, R17, R2, R3, R4, R5, R6, R7, R8, R9: footprint Resistor_SMD:R_0603_1608Metric_Pad1.05x0.95mm_HandSolder -> Resistor_SMD:R_0603_1608Metric_Pad0.98x0.95mm_HandSolder
- U1: footprint Converter_DCDC:Converter_DCDC_muRata_OKI-78SR_Horizontal -> Converter_DCDC:Converter_DCDC_Murata_OKI-78SR_Horizontal
Connections:
- IC1 pad 17: (no net) -> unconnected-(IC1-Pad17)
- IC1 pad 18: (no net) -> unconnected-(IC1-Pad18)
- IC1 pad 19: (no net) -> unconnected-(IC1-Pad19)
- IC1 pad 20: (no net) -> unconnected-(IC1-Pad20)
- IC1 pad 21: (no net) -> unconnected-(IC1-Pad21)
- IC1 pad 22: (no net) -> unconnected-(IC1-Pad22)
- IC1 pad 27: (no net) -> unconnected-(IC1-Pad27)
- IC1 pad 28: (no net) -> unconnected-(IC1-Pad28)
- IC1 pad 32: (no net) -> unconnected-(IC1-Pad32)
- IC1 pad 4: (no net) -> unconnected-(IC1-Pad4)
- IC1 pad 5: (no net) -> unconnected-(IC1-Pad5)
- IC1 pad 6: (no net) -> unconnected-(IC1-Pad6)
- IC1 pad 7: (no net) -> unconnected-(IC1-Pad7)
- U2 pad 1: Net-(U2-Pad1) -> unconnected-(U2-Pad1)
- U2 pad 13: (no net) -> unconnected-(U2-Pad13)
- U2 pad 15: (no net) -> unconnected-(U2-Pad15)
- U2 pad 16: (no net) -> unconnected-(U2-Pad16)
- U2 pad 2: (no net) -> unconnected-(U2-Pad2)
- U2 pad 4: (no net) -> unconnected-(U2-Pad4)
- U2 pad 5: (no net) -> unconnected-(U2-Pad5)
- U2 pad 6: (no net) -> unconnected-(U2-Pad6)
- U2 pad 7: (no net) -> unconnected-(U2-Pad7)
- U2 pad 8: (no net) -> unconnected-(U2-Pad8)
- U2 pad 9: Net-(U2-Pad9) -> unconnected-(U2-Pad9)
Routing:
- net unconnected-(U2-Pad1): track 0.00 -> 22.4 mm
- net Net-(U2-Pad1): track 22.4 -> 0.00 mm
- net unconnected-(U2-Pad9): track 0.00 -> 11.2 mm
- net Net-(U2-Pad9): track 11.2 -> 0.00 mm
Other:
- net class Default removed
