File: PottyBox4.kicad_sch (KiCad schematic)
At the start: 52 parts, among them IC1 ESP32-WROVER-B, J1 Sensor 1, J10 Flush 2, J2 Touch 1, J3 Sensor 2, J4 Touch 2, J5 Qwiic, J6 24VAC, J7 DEGUG, J8 Exhaust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

Commit message: Add schematic link, title block data
Other:
- title: (none) -> PottyBox4
Changed lines of the file:
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@@
 (kicad_sch (version 20210621) (generator eeschema)
   (paper "A4")
+  (title_block
+    (title "PottyBox4")
+    (date "2020-03-24")
+    (rev "1")
+  )
   (junction (at 22.86 85.09) (diameter 0) (color 0 0 0 0))
   (junction (at 25.4 67.31) (diameter 0) (color 0 0 0 0))
